File: KiCad_Project/strg+m interface.kicad_sch (KiCad schematic)
At the start: 7 parts, among them J5 AudioJack2, J6 AudioJack2

Commit message: update schematic
Connections:
- net clip_left: now also RV1.2
- net clip_right: no longer RV1.2
- net range_left: now also RV3.2
- net range_right: no longer RV3.2
Changed lines of the file:
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@@
 (kicad_sch (version 20211123) (generator eeschema)
   (paper "A5")
-  (junction (at 110.49 80.01) (diameter 0) (color 0 0 0 0)
+  (junction (at 99.695 31.75) (diameter 0) (color 0 0 0 0)
+  )
+  (junction (at 99.695 80.01) (diameter 0) (color 0 0 0 0)
+  )
+  (wire (pts (xy 97.79 31.75) (xy 99.695 31.75))
+    (stroke (width 0) (type default) (color 0 0 0 0))
   )
   (wire (pts (xy 146.05 78.105) (xy 146.05 79.375))
@@
     (stroke (width 0) (type default) (color 0 0 0 0))
   )
-  (wire (pts (xy 104.775 73.66) (xy 110.49 73.66))
+  (wire (pts (xy 99.695 80.01) (xy 100.965 80.01))
     (stroke (width 0) (type default) (color 0 0 0 0))
   )
-  (wire (pts (xy 97.79 80.01) (xy 100.965 80.01))
+  (wire (pts (xy 97.79 80.01) (xy 99.695 80.01))
     (stroke (width 0) (type default) (color 0 0 0 0))
   )
-  (wire (pts (xy 110.49 80.01) (xy 112.395 80.01))
+  (wire (pts (xy 104.775 73.66) (xy 99.695 73.66))
     (stroke (width 0) (type default) (color 0 0 0 0))
   )
@@
     (stroke (width 0) (type default) (color 0 0 0 0))
   )
-  (wire (pts (xy 110.49 80.01) (xy 108.585 80.01))
+  (wire (pts (xy 108.585 80.01) (xy 112.395 80.01))
     (stroke (width 0) (type default) (color 0 0 0 0))
   )
-  (wire (pts (xy 109.855 25.4) (xy 109.855 31.75))
+  (wire (pts (xy 104.775 25.4) (xy 99.695 25.4))
+    (stroke (width 0) (type default) (color 0 0 0 0))
+  )
+  (wire (pts (xy 99.695 31.75) (xy 100.965 31.75))
+    (stroke (width 0) (type default) (color 0 0 0 0))
+  )
+  (wire (pts (xy 99.695 25.4) (xy 99.695 31.75))
     (stroke (width 0) (type default) (color 0 0 0 0))
   )
@@
     (stroke (width 0) (type default) (color 0 0 0 0))
   )
-  (wire (pts (xy 104.775 25.4) (xy 109.855 25.4))
-    (stroke (width 0) (type default) (color 0 0 0 0))
-  )
-  (wire (pts (xy 110.49 73.66) (xy 110.49 80.01))
+  (wire (pts (xy 99.695 73.66) (xy 99.695 80.01))
     (stroke (width 0) (type default) (color 0 0 0 0))
   )
@@
     (effects (font (size 1.27 1.27)) (justify left))
   )
-  (hierarchical_label "clip_left" (shape input) (at 100.965 31.75 180)
+  (hierarchical_label "clip_left" (shape input) (at 97.79 31.75 180)
     (effects (font (size 1.27 1.27)) (justify right))
   )

Commit message: add old commits
Connections:
- net offset_left: now also RV2.3; no longer RV2.1
- net offset_right: now also RV2.1; no longer RV2.3
Other:
- moved on the sheet: RV2
Changed lines of the file:
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@@
+    (stroke (width 0) (type default) (color 0 0 0 0))
+  )
+  (wire (pts (xy 99.695 60.96) (xy 100.965 60.96))
     (stroke (width 0) (type default) (color 0 0 0 0))
   )
@@
     (stroke (width 0) (type default) (color 0 0 0 0))
   )
+  (wire (pts (xy 104.775 55.88) (xy 104.775 57.15))
+    (stroke (width 0) (type default) (color 0 0 0 0))
+  )
   (wire (pts (xy 99.695 25.4) (xy 99.695 31.75))
     (stroke (width 0) (type default) (color 0 0 0 0))
   )
   (wire (pts (xy 166.37 78.105) (xy 166.37 79.375))
+    (stroke (width 0) (type default) (color 0 0 0 0))
+  )
+  (wire (pts (xy 108.585 60.96) (xy 110.49 60.96))
     (stroke (width 0) (type default) (color 0 0 0 0))
   )
@@
     (effects (font (size 1.27 1.27)) (justify left))
   )
-  (hierarchical_label "offset_middle" (shape input) (at 104.775 57.15 90)
+  (hierarchical_label "offset_middle" (shape input) (at 104.775 55.88 90)
     (effects (font (size 1.27 1.27)) (justify left))
   )
-  (hierarchical_label "offset_left" (shape input) (at 100.965 60.96 180)
+  (hierarchical_label "offset_left" (shape input) (at 99.695 60.96 180)
     (effects (font (size 1.27 1.27)) (justify right))
   )
@@
     (effects (font (size 1.27 1.27)) (justify right))
   )
-  (hierarchical_label "offset_right" (shape input) (at 108.585 60.96 0)
+  (hierarchical_label "offset_right" (shape input) (at 110.49 60.96 0)
     (effects (font (size 1.27 1.27)) (justify left))
   )
@@
     (pin "T")
   )
-  (symbol (lib_id "Device:R_Potentiometer") (at 104.775 60.96 90) (unit 1)
+  (symbol (lib_id "Device:R_Potentiometer") (at 104.775 60.96 270) (mirror x) (unit 1)
     (in_bom yes) (on_board yes) (fields_autoplaced)
     (property "Reference" "RV2" (id 0) (at 104.775 64.77 90))
