File: KiCad_Project/strg+m main pcb.kicad_sch (KiCad schematic)
At the start: 16 parts, among them J7 Conn_02x05_Odd_Even, U1 LM324

Commit message: add old commits
Connections:
- net +12V: now also U1.4 (V+); no longer U1.11 (V-)
- net -12V: now also U1.11 (V-); no longer U1.4 (V+)
Changed lines of the file:
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@@
     (pin "2")
   )
-  (symbol (lib_id "Amplifier_Operational:LM324") (at 129.54 128.27 0) (mirror x) (unit 5)
+  (symbol (lib_id "Amplifier_Operational:LM324") (at 129.54 128.27 0) (unit 5)
     (in_bom yes) (on_board yes)
-    (property "Reference" "U1" (id 0) (at 125.73 126.9999 0)
+    (property "Reference" "U1" (id 0) (at 125.73 129.5401 0)
       (effects (font (size 1.27 1.27)) (justify right))
     )
-    (property "Value" "LM324" (id 1) (at 125.73 129.5399 0)
+    (property "Value" "LM324" (id 1) (at 125.73 127.0001 0)
       (effects (font (size 1.27 1.27)) (justify right))
     )
-    (property "Footprint" "Package_SO:SOIC-14_3.9x8.7mm_P1.27mm" (id 2) (at 128.27 130.81 0)
+    (property "Footprint" "Package_SO:SOIC-14_3.9x8.7mm_P1.27mm" (id 2) (at 128.27 125.73 0)
       (effects (font (size 1.27 1.27)) hide)
     )
-    (property "Datasheet" "http://www.ti.com/lit/ds/symlink/lm2902-n.pdf" (id 3) (at 130.81 133.35 0)
+    (property "Datasheet" "http://www.ti.com/lit/ds/symlink/lm2902-n.pdf" (id 3) (at 130.81 123.19 0)
       (effects (font (size 1.27 1.27)) hide)
     )
