File: KiCad_Project/strg+m.kicad_pcb (KiCad board)
At the start: 2 copper layers, 37.9 x 91.4 mm, 40 parts, among them J1 Conn_01x04_Female, J10 Conn_01x03_Male, J11 Conn_01x02_Male, J2 Conn_01x03_Female, J3 Conn_01x03_Female, J4 Conn_01x02_Female, J5 AudioJack2, J6 AudioJack2, J7 Conn_02x05_Odd_Even, J8 Conn_01x04_Male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

Commit message: update pcb layout
Connections:
- net /ctrl+m interface/0V renamed /strg+m interface/0V
- net /ctrl+m interface/cv_in renamed /strg+m interface/cv_in
- net /ctrl+m interface/cv_out renamed /strg+m interface/cv_out
- net /ctrl+m interface/neg_halfwave renamed /strg+m interface/neg_halfwave
- net /ctrl+m interface/offset_left renamed /strg+m interface/offset_left
- net /ctrl+m interface/offset_middle renamed /strg+m interface/offset_middle
- net /ctrl+m interface/offset_right renamed /strg+m interface/offset_right
- net /ctrl+m interface/pos_halfwave renamed /strg+m interface/pos_halfwave
- net /ctrl+m main pcb/clip_left renamed /strg+m main pcb/clip_left
- net /ctrl+m main pcb/clip_right renamed /strg+m main pcb/clip_right
- net /ctrl+m main pcb/cv_in renamed /strg+m main pcb/cv_in
- net /ctrl+m main pcb/cv_out renamed /strg+m main pcb/cv_out
- net /ctrl+m main pcb/neg_halfwave renamed /strg+m main pcb/neg_halfwave
- net /ctrl+m main pcb/offset_left renamed /strg+m main pcb/offset_left
- net /ctrl+m main pcb/offset_middle renamed /strg+m main pcb/offset_middle
- net /ctrl+m main pcb/offset_right renamed /strg+m main pcb/offset_right
- net /ctrl+m main pcb/pos_halfwave renamed /strg+m main pcb/pos_halfwave
- net /ctrl+m main pcb/range_left renamed /strg+m main pcb/range_left
- J1 pad 2: /ctrl+m interface/range_left -> /strg+m interface/range_left
- J1 pad 3: /ctrl+m interface/range_right -> /strg+m interface/range_right
- J4 pad 1: /ctrl+m interface/clip_left -> /strg+m interface/clip_left
- J4 pad 2: /ctrl+m interface/clip_right -> /strg+m interface/clip_right
- RV1 pad 1: /ctrl+m interface/clip_left -> /strg+m interface/clip_left
- RV1 pad 2: /ctrl+m interface/clip_right -> /strg+m interface/clip_left
- RV1 pad 3: /ctrl+m interface/clip_right -> /strg+m interface/clip_right
- RV3 pad 1: /ctrl+m interface/range_left -> /strg+m interface/range_left
- RV3 pad 2: /ctrl+m interface/range_right -> /strg+m interface/range_left
- RV3 pad 3: /ctrl+m interface/range_right -> /strg+m interface/range_right
Routing:
- net /ctrl+m interface/range_right: track 20.3 -> 0.00 mm
- net /strg+m interface/range_left: track 0.00 -> 19.5 mm
- net /ctrl+m interface/range_left: track 17.8 -> 0.00 mm
- net /strg+m interface/range_right: track 0.00 -> 17.8 mm
- net /strg+m interface/clip_right: track 0.00 -> 8.90 mm
- net /ctrl+m interface/clip_right: track 8.90 -> 0.00 mm
- net /strg+m interface/clip_left: track 0.00 -> 5.34 mm
- net /ctrl+m interface/clip_left: track 2.84 -> 0.00 mm
- net /strg+m interface/pos_halfwave: track 23.9 -> 24.4 mm

Commit message: add old commits
Connections:
- RV2 pad 1: /strg+m interface/offset_left -> /strg+m interface/offset_right
- RV2 pad 3: /strg+m interface/offset_right -> /strg+m interface/offset_left
- U1 pad 11: +12V -> -12V
- U1 pad 4: -12V -> +12V
Routing:
- net /strg+m interface/offset_left: track 3.17 -> 11.3 mm
- net /strg+m interface/offset_right: track 3.18 -> 6.36 mm
Changed lines of the file:
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@@
     (pad "" np_thru_hole circle (at 7 1.9 90) (size 4 4) (drill 2) (layers *.Cu *.Mask))
     (pad "1" thru_hole circle (at 0 0 90) (size 1.8 1.8) (drill 1) (layers *.Cu *.Mask)
-      (net 16 "/strg+m interface/offset_left") (pinfunction "1") (pintype "passive"))
+      (net 18 "/strg+m interface/offset_right") (pinfunction "1") (pintype "passive"))
     (pad "2" thru_hole circle (at 0 -2.5 90) (size 1.8 1.8) (drill 1) (layers *.Cu *.Mask)
       (net 17 "/strg+m interface/offset_middle") (pinfunction "2") (pintype "passive"))
     (pad "3" thru_hole circle (at 0 -5 90) (size 1.8 1.8) (drill 1) (layers *.Cu *.Mask)
-      (net 18 "/strg+m interface/offset_right") (pinfunction "3") (pintype "passive"))
+      (net 16 "/strg+m interface/offset_left") (pinfunction "3") (pintype "passive"))
     (model "${KICAD6_3RD_PARTY}/Potentiometer/RK097.step"
       (offset (xyz 0 0 0))
@@
       (net 28 "/strg+m main pcb/offset_middle") (pinfunction "+") (pintype "input"))
     (pad "4" smd roundrect (at -2.475 0) (size 1.95 0.6) (layers "B.Cu" "B.Paste" "B.Mask") (roundrect_rratio 0.25)
-      (net 3 "-12V") (pinfunction "V+") (pintype "power_in"))
+      (net 2 "+12V") (pinfunction "V+") (pintype "power_in"))
     (pad "5" smd roundrect (at -2.475 -1.27) (size 1.95 0.6) (layers "B.Cu" "B.Paste" "B.Mask") (roundrect_rratio 0.25)
       (net 4 "/strg+m main pcb/clip_right") (pinfunction "+") (pintype "input"))
@@
       (net 1 "GND") (pinfunction "+") (pintype "input"))
     (pad "11" smd roundrect (at 2.475 0) (size 1.95 0.6) (layers "B.Cu" "B.Paste" "B.Mask") (roundrect_rratio 0.25)
-      (net 2 "+12V") (pinfunction "V-") (pintype "power_in"))
+      (net 3 "-12V") (pinfunction "V-") (pintype "power_in"))
     (pad "12" smd roundrect (at 2.475 1.27) (size 1.95 0.6) (layers "B.Cu" "B.Paste" "B.Mask") (roundrect_rratio 0.25)
       (net 9 "Net-(D4-Pad2)") (pinfunction "+") (pintype "input"))
@@
   (segment (start -1.28 -90.17) (end -1.28 -74.118) (width 0.25) (layer "F.Cu") (net 15))
   (segment (start -1.28 -74.118) (end -2.5 -72.898) (width 0.25) (layer "F.Cu") (net 15))
-  (segment (start 2.5 -47.015) (end 2.525 -46.99) (width 0.25) (layer "B.Cu") (net 16))
-  (segment (start 2.5 -50.15) (end 2.5 -47.015) (width 0.25) (layer "B.Cu") (net 16))
-  (segment (start 0 -47.005) (end -0.015 -46.99) (width 0.25) (layer "B.Cu") (net 17))
-  (segment (start 0 -50.15) (end 0 -47.005) (width 0.25) (layer "B.Cu") (net 17))
-  (segment (start -2.5 -47.045) (end -2.555 -46.99) (width 0.25) (layer "B.Cu") (net 18))
-  (segment (start -2.5 -50.15) (end -2.5 -47.045) (width 0.25) (layer "B.Cu") (net 18))
+  (segment (start -1.300489 -51.349511) (end 3.260489 -51.349511) (width 0.2) (layer "F.Cu") (net 16))
+  (segment (start 3.260489 -51.349511) (end 3.699511 -50.910489) (width 0.2) (layer "F.Cu") (net 16))
+  (segment (start 3.699511 -48.164511) (end 2.525 -46.99) (width 0.2) (layer "F.Cu") (net 16))
+  (segment (start 3.699511 -50.910489) (end 3.699511 -48.164511) (width 0.2) (layer "F.Cu") (net 16))
+  (segment (start -2.5 -50.15) (end -1.300489 -51.349511) (width 0.2) (layer "F.Cu") (net 16))
+  (segment (start 0 -47.005) (end -0.015 -46.99) (width 0.2) (layer "B.Cu") (net 17))
+  (segment (start 0 -50.15) (end 0 -47.005) (width 0.2) (layer "B.Cu") (net 17))
+  (segment (start 2.5 -50.15) (end 1.245 -48.895) (width 0.2) (layer "F.Cu") (net 18))
+  (segment (start 1.245 -48.895) (end -0.65 -48.895) (width 0.2) (layer "F.Cu") (net 18))
+  (segment (start -0.65 -48.895) (end -2.555 -46.99) (width 0.2) (layer "F.Cu") (net 18))
   (segment (start -0.015 -19.66) (end 0 -19.645) (width 0.25) (layer "F.Cu") (net 19))
   (segment (start -0.015 -24.13) (end -0.015 -19.66) (width 0.25) (layer "F.Cu") (net 19))
